File: board/power-board.brd (EAGLE design)
At the start: 95.9 x 90.2 mm, 447 parts, among them J1 H1, J2 H2, J6 DF13-8P-1.25DS, J7 DF13-10P-1.25DS, J8 DF13-4P-1.25DS, J9 DF13-4P-1.25DS, Q3 SI7288, U1 INA214DCK, U10 INA214DCK, U11 INA214DCK, U12 INA214DCK, U13 MCP6561T-E/LT, U14 INA214DCK, U15 SN74AUP1G00DCK, U16 SN74LVC1G373DCK, U17 NTHD4508NT1, U18 MCP6561T-E/LT, U19 INA214DCK, U2 INA214DCK, U20 SN74AUP1G00DCK, U21 SN74LVC1G373DCK, U22 NTHD4508NT1, U23 MCP6561T-E/LT, U24 INA214DCK, U25 SN74AUP1G00DCK, U26 SN74LVC1G373DCK, U27 NTHD4508NT1, U28 MCP6561T-E/LT, U29 INA214DCK, U3 INA214DCK, U30 SN74AUP1G00DCK, U31 SN74LVC1G373DCK, U32 NTHD4508NT1, U33 MCP6561T-E/LT, U34 INA214DCK, U35 SN74AUP1G00DCK, U36 SN74LVC1G373DCK, U37 NTHD4508NT1, U38 MCP6561T-E/LT, U39 INA214DCK, U4 INA214DCK, U40 SN74AUP1T08DCK, U41 SN74LVC1G373DCK, U42 FDS8858CZ, U43 TLV3491AIDBV, U44 TPS62132RGT, U45 FDS8858CZ, U46 TLV3491AIDBV, U47 TPS62133RGT, U48 FDS8858CZ, U49 MSP430F2132, U5 INA214DCK, U50 ADG732, U51 SPV1040T, U52 SPV1040T, U53 BQ24650_RVA_16, U54 INA214DCK, U55 SPV1040T, U56 SPV1040T, U57 SPV1040T, U58 SPV1040T, U6 INA214DCK, U7 INA214DCK, U8 INA214DCK, U9 INA214DCK, X1 32.768k

Commit message: no airwires
Parts:
- removed TP28, TP30, TP34, TP36: PTR1TP09R, testpad:TP09R
- moved TP35 121.3 mm to (18.3, 1.83)
- moved TP29 95.5 mm to (14.6, 1.83)
- moved TP33 23.7 mm to (22.6, 1.83)
- moved TP31 17.8 mm to (10.4, 1.83)
- moved TP32 17.6 mm to (16.5, 1.83)
- moved R26 12.8 mm to (30.5, 16.5), turned to 180 degrees
- moved C26 11.0 mm to (30.5, 27.4)
- moved R25 11.0 mm to (30.5, 20.1)
- moved R27 11.0 mm to (30.5, 31.1)
- moved R28 11.0 mm to (30.5, 29.3)
- moved C25 9.14 mm to (30.5, 18.3), turned to 0 degrees
- moved C6 0.61 mm to (40.2, 71.3)
- moved L7 0.45 mm to (28.7, 9.75)
- moved L9 0.45 mm to (28.7, 50.0)
- moved L3 0.39 mm to (28.7, 39.6)
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Connections:
- net CHARGE_IN: no longer TP28.TP, TP34.TP
- net GND: no longer TP30.TP, TP36.TP
- net MPPT2L_PV_P: no longer R27.2
- net MPPT2_MID: now also R27.2
Routing:
- net MPPT3_MID: track 147.3 -> 204.2 mm, vias 24 -> 25
- net MPPT2_MID: track 196.0 -> 237.8 mm, vias 21 -> 22
- net MPPT1_MID: track 165.2 -> 200.6 mm, vias 28 -> 29
- net CHARGE_IN: track 202.6 -> 230.6 mm, vias 8 -> 10
- net MPPT2L_PV_P: track 93.7 -> 105.7 mm
- net MPPT2_MID_PV_VSENSE: track 13.1 -> 18.3 mm
- net MPPT2_LOWER_PV_VSENSE: track 18.0 -> 12.8 mm
- net MPPT_BUS_VSENSE: track 16.3 -> 14.6 mm
- net MPPT1L_PV_P: track 153.0 -> 151.6 mm, vias 8 -> 7
- net GND: track 498.7 -> 500.0 mm, vias 255 -> 256
- net N$794: track 11.9 -> 10.9 mm
- net UVP3V3_OUT: track 283.1 -> 284.0 mm
- net MPPT1H_PV_P: track 143.9 -> 144.7 mm
- net MPPT3L_PV_P: track 104.0 -> 104.7 mm
Other:
- board text added: "1"
- board text added: "1H"
- board text added: "1L"
- board text added: "2"
- board text added: "2H"
- board text added: "2L"
- board text added: "3"
- board text added: "3H"
- board text added: "3L"
- board text added: "GND"
- board text added: "H"
- board text added: "L"
- board text added: "MID"
- board text added: "MPPT OUT"
- board text added: "PV EAST"
- board text added: "PV NORTH"
- board text added: "PV SOUTH"
- board text added: "PV TOP"
- board text added: "PV WEST"
- board text removed: "0V"
- board text removed: "CHG IN"
- board text removed: "E1C"
- board text removed: "E2C"
- board text removed: "MPPT1"
- board text removed: "MPPT2"
- board text removed: "MPPT2_OUT"
- board text removed: "MPPT2_PV_P"
- board text removed: "N1C"
- board text removed: "S1C"
- board text removed: "S2C"
- board text removed: "W1C"
- board text removed: "W2C"
