File: board/power-board.brd (EAGLE design)
At the start: 95.9 x 90.2 mm, 445 parts, among them J1 H1, J2 H2, J6 DF13-8P-1.25DS, J7 DF13-10P-1.25DS, J8 DF13-4P-1.25DS, J9 DF13-4P-1.25DS, Q3 SI7288, U1 INA214DCK, U10 INA214DCK, U11 INA214DCK, U12 INA214DCK, U13 MCP6561T-E/LT, U14 INA214DCK, U15 SN74AUP1G00DCK, U16 SN74LVC1G373DCK, U17 NTHD4508NT1, U18 MCP6561T-E/LT, U19 INA214DCK, U2 INA214DCK, U20 SN74AUP1G00DCK, U21 SN74LVC1G373DCK, U22 NTHD4508NT1, U23 MCP6561T-E/LT, U24 INA214DCK, U25 SN74AUP1G00DCK, U26 SN74LVC1G373DCK, U27 NTHD4508NT1, U28 MCP6561T-E/LT, U29 INA214DCK, U3 INA214DCK, U30 SN74AUP1G00DCK, U31 SN74LVC1G373DCK, U32 NTHD4508NT1, U33 MCP6561T-E/LT, U34 INA214DCK, U35 SN74AUP1G00DCK, U36 SN74LVC1G373DCK, U37 NTHD4508NT1, U38 MCP6561T-E/LT, U39 INA214DCK, U4 INA214DCK, U40 SN74AUP1T08DCK, U41 SN74LVC1G373DCK, U42 FDS8858CZ, U43 TLV3491AIDBV, U44 TPS62132RGT, U45 FDS8858CZ, U46 TLV3491AIDBV, U47 TPS62133RGT, U48 FDS8858CZ, U49 MSP430F2132, U5 INA214DCK, U50 ADG732, U51 SPV1040T, U52 SPV1040T, U53 BQ24650_RVA_16, U54 INA214DCK, U55 SPV1040T, U56 SPV1040T, U57 SPV1040T, U58 SPV1040T, U6 INA214DCK, U7 INA214DCK, U8 INA214DCK, U9 INA214DCK, X1 32.768k

Commit message: updating component values (fixing prev errors)
Parts:
- R102, R95: value 20k -> 14.5k
- U13, U18, U23, U28, U33, U38: value MCP6561T-E/LT -> MCP6561R
Changed lines of the file:
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@@
 <?xml version="1.0" encoding="utf-8"?>
 <!DOCTYPE eagle SYSTEM "eagle.dtd">
-<eagle version="6.6.0">
+<eagle version="9.0.1">
 <drawing>
 <settings>
 <setting alwaysvectorfont="no"/>
+<setting keepoldvectorfont="yes"/>
 <setting verticaltext="up"/>
 </settings>
 <grid distance="24" unitdist="mil" unit="mil" style="lines" multiple="1" display="yes" altdistance="2" altunitdist="mil" altunit="mil"/>
 <layers>
-<layer number="1" name="Top" color="4" fill="1" visible="no" active="yes"/>
-<layer number="2" name="Route2" color="5" fill="5" visible="no" active="yes"/>
+<layer number="1" name="Top" color="4" fill="1" visible="yes" active="yes"/>
+<layer number="2" name="Route2" color="5" fill="5" visible="yes" active="yes"/>
 <layer number="3" name="Route3" color="4" fill="3" visible="no" active="no"/>
 <layer number="4" name="Route4" color="1" fill="4" visible="no" active="no"/>
@@
 <layer number="20" name="Dimension" color="15" fill="1" visible="yes" active="yes"/>
 <layer number="21" name="tPlace" color="7" fill="1" visible="no" active="yes"/>
-<layer number="22" name="bPlace" color="7" fill="1" visible="yes" active="yes"/>
+<layer number="22" name="bPlace" color="7" fill="1" visible="no" active="yes"/>
 <layer number="23" name="tOrigins" color="15" fill="1" visible="no" active="yes"/>
-<layer number="24" name="bOrigins" color="15" fill="1" visible="yes" active="yes"/>
+<layer number="24" name="bOrigins" color="15" fill="1" visible="no" active="yes"/>
 <layer number="25" name="tNames" color="7" fill="1" visible="no" active="yes"/>
-<layer number="26" name="bNames" color="7" fill="1" visible="yes" active="yes"/>
+<layer number="26" name="bNames" color="7" fill="1" visible="no" active="yes"/>
 <layer number="27" name="tValues" color="7" fill="1" visible="no" active="yes"/>
 <layer number="28" name="bValues" color="7" fill="1" visible="no" active="yes"/>
 <layer number="29" name="tStop" color="7" fill="3" visible="no" active="yes"/>
-<layer number="30" name="bStop" color="7" fill="6" visible="yes" active="yes"/>
+<layer number="30" name="bStop" color="7" fill="6" visible="no" active="yes"/>
 <layer number="31" name="tCream" color="7" fill="4" visible="no" active="yes"/>
 <layer number="32" name="bCream" color="7" fill="5" visible="no" active="yes"/>
@@
 <param name="dpMaxLengthDifference" value="10mm"/>
 <param name="dpGapFactor" value="2.5"/>
-<param name="checkGrid" value="0"/>
 <param name="checkAngle" value="0"/>
 <param name="checkFont" value="1"/>
 <param name="checkRestrict" value="1"/>
+<param name="checkStop" value="0"/>
+<param name="checkValues" value="0"/>
 <param name="useDiameter" value="13"/>
 <param name="maxErrors" value="50"/>
@@
 <pass name="Default">
 <param name="RoutingGrid" value="6.25mil"/>
+<param name="AutoGrid" value="1"/>
+<param name="Efforts" value="0"/>
+<param name="TopRouterVariant" value="1"/>
 <param name="tpViaShape" value="round"/>
 <param name="PrefDir.1" value="*"/>
@@
 <attribute name="NAME" x="68.453" y="19.4945" size="0.8128" layer="26" font="vector" ratio="14" rot="MR0"/>
 </element>
-<element name="U13" library="tomparts" package="SOT23-5" value="MCP6561T-E/LT" x="39.37" y="16.0655" smashed="yes" rot="MR0">
+<element name="U13" library="tomparts" package="SOT23-5" value="MCP6561R" x="39.37" y="16.0655" smashed="yes" rot="MR0">
 <attribute name="NAME" x="40.5765" y="18.415" size="0.8128" layer="26" font="vector" ratio="14" rot="MR0"/>
 </element>
@@
 <attribute name="NAME" x="47.1297" y="53.2003" size="0.8128" layer="25" font="vector" ratio="14"/>
 </element>
-<element name="R95" library="rcl" package="R0603" value="20k" x="44.9199" y="60.5028" smashed="yes">
+<element name="R95" library="rcl" package="R0603" value="14.5k" x="44.9199" y="60.5028" smashed="yes">
 <attribute name="NAME" x="43.9801" y="61.4426" size="0.8128" layer="25" font="vector" ratio="14"/>
 </element>
@@
 <attribute name="NAME" x="73.3933" y="73.1139" size="0.8128" layer="25" font="vector" ratio="14"/>
 </element>
-<element name="R102" library="rcl" package="R0603" value="20k" x="78.9432" y="67.4751" smashed="yes" rot="R90">
+<element name="R102" library="rcl" package="R0603" value="14.5k" x="78.9432" y="67.4751" smashed="yes" rot="R90">
 <attribute name="NAME" x="80.645" y="65.9257" size="0.8128" layer="25" font="vector" ratio="14" rot="R90"/>
 </element>
@@
 <attribute name="NAME" x="68.453" y="29.1973" size="0.8128" layer="26" font="vector" ratio="14" rot="MR0"/>
 </element>
-<element name="U18" library="tomparts" package="SOT23-5" value="MCP6561T-E/LT" x="39.37" y="25.9715" smashed="yes" rot="MR0">
+<element name="U18" library="tomparts" package="SOT23-5" value="MCP6561R" x="39.37" y="25.9715" smashed="yes" rot="MR0">
 <attribute name="NAME" x="40.5765" y="28.321" size="0.8128" layer="26" font="vector" ratio="14" rot="MR0"/>
 </element>
@@
 <attribute name="NAME" x="68.0466" y="39.3065" size="0.8128" layer="26" font="vector" ratio="14" rot="MR0"/>
 </element>
-<element name="U23" library="tomparts" package="SOT23-5" value="MCP6561T-E/LT" x="39.37" y="35.8775" smashed="yes" rot="MR0">
+<element name="U23" library="tomparts" package="SOT23-5" value="MCP6561R" x="39.37" y="35.8775" smashed="yes" rot="MR0">
 <attribute name="NAME" x="40.5765" y="38.227" size="0.8128" layer="26" font="vector" ratio="14" rot="MR0"/>
 </element>
@@
 <attribute name="NAME" x="68.453" y="49.5173" size="0.8128" layer="26" font="vector" ratio="14" rot="MR0"/>
 </element>
-<element name="U28" library="tomparts" package="SOT23-5" value="MCP6561T-E/LT" x="39.37" y="45.7835" smashed="yes" rot="MR0">
+<element name="U28" library="tomparts" package="SOT23-5" value="MCP6561R" x="39.37" y="45.7835" smashed="yes" rot="MR0">
 <attribute name="NAME" x="40.5765" y="48.133" size="0.8128" layer="26" font="vector" ratio="14" rot="MR0"/>
 </element>
@@
 <attribute name="NAME" x="68.1482" y="59.1185" size="0.8128" layer="26" font="vector" ratio="14" rot="MR0"/>
 </element>
-<element name="U33" library="tomparts" package="SOT23-5" value="MCP6561T-E/LT" x="39.37" y="55.6895" smashed="yes" rot="MR0">
+<element name="U33" library="tomparts" package="SOT23-5" value="MCP6561R" x="39.37" y="55.6895" smashed="yes" rot="MR0">
 <attribute name="NAME" x="40.5765" y="58.039" size="0.8128" layer="26" font="vector" ratio="14" rot="MR0"/>
 </element>
@@
 <attribute name="NAME" x="68.453" y="69.0245" size="0.8128" layer="26" font="vector" ratio="14" rot="MR0"/>
 </element>
-<element name="U38" library="tomparts" package="SOT23-5" value="MCP6561T-E/LT" x="39.37" y="65.5955" smashed="yes" rot="MR0">
+<element name="U38" library="tomparts" package="SOT23-5" value="MCP6561R" x="39.37" y="65.5955" smashed="yes" rot="MR0">
 <attribute name="NAME" x="40.5765" y="67.945" size="0.8128" layer="26" font="vector" ratio="14" rot="MR0"/>
 </element>
